Commit message: Dex wrist update

File: xacro_files_backup/launch/stretch_description/urdf/stretch.urdf (robot description, URDF)
Before this commit: robot stretch_description, 46 links, 45 joints
Links:
- added link camera_accel_frame
- added link camera_accel_optical_frame
- added link camera_gyro_frame
- added link camera_gyro_optical_frame
- added link caster_link, mass 0.01; collision sphere radius=0.032; visual mesh filename=package://stretch_description/meshes/omni_wheel_m.STL
- added link link_grasp_center
- link electrode1: geometry visual sphere radius=0.01
- link electrode2: geometry visual sphere radius=0.01
- link electrode3: geometry visual sphere radius=0.01
- link electrode4: geometry visual sphere radius=0.01
- link electrode5: geometry visual sphere radius=0.01
- link electrode6: geometry visual sphere radius=0.01
- link link_aruco_inner_wrist: mass 0.000225 -> 0.0
- link link_aruco_shoulder: mass 0.000399141592654 -> 0.0
- link link_aruco_top_wrist: mass 0.000225 -> 0.0
- link link_left_wheel: mass 0.00356714564938 -> 0.01
- link link_right_wheel: mass 0.00356714564938 -> 0.01
Joints:
- added joint camera_accel_joint: type fixed, parent camera_link, child camera_accel_frame, origin xyz=-0.01174 -0.00552 0.0051 rpy=0.0 0.0 0.0
- added joint camera_accel_optical_joint: type fixed, parent camera_accel_frame, child camera_accel_optical_frame, origin xyz=0.0 0.0 0.0 rpy=-1.57079632679 0.0 -1.57079632679
- added joint camera_gyro_joint: type fixed, parent camera_link, child camera_gyro_frame, origin xyz=-0.01174 -0.00552 0.0051 rpy=0.0 0.0 0.0
- added joint camera_gyro_optical_joint: type fixed, parent camera_gyro_frame, child camera_gyro_optical_frame, origin xyz=0.0 0.0 0.0 rpy=-1.57079632679 0.0 -1.57079632679
- added joint caster_joint: type fixed, parent base_link, child caster_link, origin xyz=-0.245 0.0 0.032 rpy=-1.57079632679 0.0 0.0, axis 0.0 0.0 1.0
- added joint joint_grasp_center: type fixed, parent link_straight_gripper, child link_grasp_center, origin xyz=0.0 -0.0125 0.23 rpy=0.0 0.0 3.141579
- joint center_to_tool: axis 0.0 0.0 0.0 -> (none); origin xyz=-0.05 0.055 0.15 rpy=1.57079632679 2.09439510239 0 -> xyz=0.0 0.055 0.0 rpy=1.57079632679 3.141579 0.0; parent link_gripper_fingertip_left -> link_grasp_center
- joint root_to_electrode1: origin xyz=0.015 0.075 0 rpy=0 0 0 -> xyz=-0.055 -0.035 0.01 rpy=0.0 0.0 0.0
- joint root_to_electrode2: origin xyz=0.015 0.145 0 rpy=0 0 0 -> xyz=-0.055 0.035 0.01 rpy=0.0 0.0 0.0
- joint root_to_electrode3: origin xyz=0.070 0.075 0 rpy=0 0 0 -> xyz=0.0 -0.035 0.01 rpy=0.0 0.0 0.0
- joint root_to_electrode4: origin xyz=0.070 0.145 0 rpy=0 0 0 -> xyz=0.0 0.035 0.01 rpy=0.0 0.0 0.0
- joint root_to_electrode5: origin xyz=0.125 0.075 0 rpy=0 0 0 -> xyz=0.055 -0.035 0.01 rpy=0.0 0.0 0.0
- joint root_to_electrode6: origin xyz=0.125 0.145 0 rpy=0 0 0 -> xyz=0.055 0.035 0.01 rpy=0.0 0.0 0.0

File: xacro_files_backup/launch/stretch_description/urdf/stretch_description.xacro (robot description, xacro)
@@ -1,5 +1,6 @@
 <?xml version="1.0"?>
 <robot xmlns:xacro="http://www.ros.org/wiki/xacro" name="stretch">
-  <xacro:include filename="stretch_gripper.xacro" />
+  <xacro:include filename="stretch_dex_wrist.xacro" />
+  <!-- <xacro:include filename="stretch_gripper.xacro" /> -->
   <!--<xacro:include filename="stretch_gripper_with_puller.xacro" />-->
   <!--<xacro:include filename="stretch_dry_erase_marker.xacro" />-->

File: xacro_files_backup/launch/stretch_description/urdf/stretch_gripper.xacro (robot description, xacro)
@@ -285,3 +285,204 @@
       link="link_grasp_center" />
   </joint>
+<!-- wash tool begins -->
+  <link name="root_tool">
+    <inertial>
+      <origin rpy="0.0 0.0 0.0" xyz="0.0 0.0 0.03"/>
+      <mass value="0.1"/>
+      <inertia ixx="0.01" ixy="0.0" ixz="0.0" iyy="0.01" iyz="0.0" izz="0.01"/>
+    </inertial>
+    <visual>
+      <origin rpy="0 0 0" xyz="0 0.06 0"/>
+      <!-- xyz -0.1 0.050 0.1 -->
+      <!-- <origin rpy="1.57079632679 0 0" xyz="0.190596948564 -0.015 0.0"/> -->
+      <geometry>
+        <!-- <mesh filename="package://stretch_description/meshes/base_link.STL" scale="1 1 1"/> -->
+        <mesh filename="package://stretch_description/meshes/Tool1.STL" scale="0.01 0.01 0.01"/>
+        <!-- <mesh filename="package://stretch_description/meshes/Tool1-3.0.stl" scale="0.01 0.01 0.01"/> -->
+        <!-- <mesh filename="package://stretch_description/meshes/Tool1-3.0.stl" scale="0.01 0.01 0.01"/> -->
+        <!-- package://stretch_description/meshes/link_wrist_yaw_bottom.STL" -->
+      </geometry>
+    </visual>
+    <collision>
+      <origin rpy="0 0 0" xyz="0 0.06 0"/>
+      <geometry>
+        <mesh filename="package://stretch_description/meshes/Tool1.STL" scale="0.01 0.01 0.01"/>
+      </geometry>
+    </collision>
+  </link>
+  <joint name="center_to_tool" type="fixed">
+    <origin rpy="0 0 1.57079632679" xyz="0.108 -0.07 -0.055"/>
+    <parent link="link_grasp_center"/>
+    <child link="root_tool"/>
+    <!-- <origin rpy="1.57079632679 2.09439510239 0" xyz="-0.05 0.055 0.15"/> -->
+    <!-- 1.5708 -1.5615 3.1416 -->
+    <!-- 1.57079632679 4.51275387511e-14 2.60113659716 -->
+    <!-- 0.190596948564 -0.015 0.0 -->
+    <!-- <axis xyz="0.0 0.0 0.0"/>
+    <parent link="link_gripper_fingertip_left"/>
+    <child link="root_tool"/> -->
+  </joint>
+  <link name="electrode1">
+    <visual>
+      <geometry>
+        <sphere radius="0.01"/>
+      </geometry>
+      <material name="green">
+        <color rgba="0 1 0 1"/>
+      </material>
+      <!-- <origin rpy="0 0 0" xyz="0.5 0.5 0"/> -->
+      <!-- <material name="blue"/> -->
+    </visual>
+    <collision>
+      <origin rpy="0 0 0" xyz="0 0.06 0"/>
+      <geometry>
+        <sphere radius="0.01"/>
+      </geometry>
+    </collision>
+  </link>
+  <joint name="root_to_electrode1" type="prismatic">
+    <origin rpy="0 0 0" xyz="0.015 0.075 0"/>
+    <parent link="root_tool"/>
+    <child link="electrode1"/>
+    <axis xyz="0.0 0.0 1.0"/>
+    <limit effort="100.0" lower="0.0" upper="1.1" velocity="1.0"/>
+    <!-- <origin xyz="0 -0.22 0.25"/> -->
+    <!-- 0.035 -0.05 -0.05 -->
+  </joint>
+  <link name="electrode2">
+    <visual>
+      <geometry>
+        <sphere radius="0.01"/>
+      </geometry>
+      <material name="green">
+        <color rgba="0 1 0 1"/>
+      </material>
+      <!-- <origin rpy="0 0 0" xyz="0.5 0.5 0"/> -->
+      <!-- <material name="blue"/> -->
+    </visual>
+    <collision>
+      <origin rpy="0 0 0" xyz="0 0.06 0"/>
+      <geometry>
+        <sphere radius="0.01"/>
+      </geometry>
+    </collision>
+  </link>
+  <joint name="root_to_electrode2" type="prismatic">
+    <origin rpy="0 0 0" xyz="0.015 0.145 0"/>
+    <parent link="root_tool"/>
+    <child link="electrode2"/>
+    <axis xyz="0.0 0.0 1.0"/>
+    <limit effort="100.0" lower="0.0" upper="1.1" velocity="1.0"/>
+    <!-- <origin xyz="0 -0.22 0.25"/> -->
+    <!-- 0.035 -0.05 -0.05 -->
+  </joint>
+  <link name="electrode3">
+    <visual>
+      <geometry>
+        <sphere radius="0.01"/>
+      </geometry>
+      <material name="green">
+        <color rgba="0 1 0 1"/>
+      </material>
+      <!-- <origin rpy="0 0 0" xyz="0.5 0.5 0"/> -->
+      <!-- <material name="blue"/> -->
+    </visual>
+    <collision>
+      <origin rpy="0 0 0" xyz="0 0.06 0"/>
+      <geometry>
+        <sphere radius="0.01"/>
+      </geometry>
+    </collision>
+  </link>
+  <joint name="root_to_electrode3" type="prismatic">
+    <origin rpy="0 0 0" xyz="0.070 0.075 0"/>
+    <parent link="root_tool"/>
+    <child link="electrode3"/>
+    <axis xyz="0.0 0.0 1.0"/>
+    <limit effort="100.0" lower="0.0" upper="1.1" velocity="1.0"/>
+    <!-- <origin xyz="0 -0.22 0.25"/> -->
+    <!-- 0.035 -0.05 -0.05 -->
+  </joint>
+  <link name="electrode4">
+    <visual>
+      <geometry>
+        <sphere radius="0.01"/>
+      </geometry>
+      <material name="green">
+        <color rgba="0 1 0 1"/>
+      </material>
+      <!-- <origin rpy="0 0 0" xyz="0.5 0.5 0"/> -->
+      <!-- <material name="blue"/> -->
+    </visual>
+    <collision>
+      <origin rpy="0 0 0" xyz="0 0.06 0"/>
+      <geometry>
+        <sphere radius="0.01"/>
+      </geometry>
+    </collision>
+  </link>
+  <joint name="root_to_electrode4" type="prismatic">
+    <origin rpy="0 0 0" xyz="0.070 0.145 0"/>
+    <parent link="root_tool"/>
+    <child link="electrode4"/>
+    <axis xyz="0.0 0.0 1.0"/>
+    <limit effort="100.0" lower="0.0" upper="1.1" velocity="1.0"/>
+    <!-- <origin xyz="0 -0.22 0.25"/> -->
+    <!-- 0.035 -0.05 -0.05 -->
+  </joint>
+  <link name="electrode5">
+    <visual>
+      <geometry>
+        <sphere radius="0.01"/>
+      </geometry>
+      <material name="green">
+        <color rgba="0 1 0 1"/>
+      </material>
+      <!-- <origin rpy="0 0 0" xyz="0.5 0.5 0"/> -->
+      <!-- <material name="blue"/> -->
+    </visual>
+    <collision>
+      <origin rpy="0 0 0" xyz="0 0.06 0"/>
+      <geometry>
+        <sphere radius="0.01"/>
+      </geometry>
+    </collision>
+  </link>
+  <joint name="root_to_electrode5" type="prismatic">
+    <origin rpy="0 0 0" xyz="0.125 0.075 0"/>
+    <parent link="root_tool"/>
+    <child link="electrode5"/>
+    <axis xyz="0.0 0.0 1.0"/>
+    <limit effort="100.0" lower="0.0" upper="1.1" velocity="1.0"/>
+    <!-- <origin xyz="0 -0.22 0.25"/> -->
+    <!-- 0.035 -0.05 -0.05 -->
+  </joint>
+  <link name="electrode6">
+    <visual>
+      <geometry>
+        <sphere radius="0.01"/>
+      </geometry>
+      <material name="green">
+        <color rgba="0 1 0 1"/>
+      </material>
+      <!-- <origin rpy="0 0 0" xyz="0.5 0.5 0"/> -->
+      <!-- <material name="blue"/> -->
+    </visual>
+    <collision>
+      <origin rpy="0 0 0" xyz="0 0.06 0"/>
+      <geometry>
+        <sphere radius="0.01"/>
+      </geometry>
+    </collision>
+  </link>
+  <joint name="root_to_electrode6" type="prismatic">
+    <origin rpy="0 0 0" xyz="0.125 0.145 0"/>
+    <parent link="root_tool"/>
+    <child link="electrode6"/>
+    <axis xyz="0.0 0.0 1.0"/>
+    <limit effort="100.0" lower="0.0" upper="1.1" velocity="1.0"/>
+    <!-- <origin xyz="0 -0.22 0.25"/> -->
+    <!-- 0.035 -0.05 -0.05 -->
+  </joint>
+  <!-- wash tool ends -->
 </robot>

File: xacro_files_backup/launch/stretch_description/urdf/stretch_uncalibrated.urdf (robot description, URDF)
Before this commit: robot stretch, 43 links, 42 joints
Links:
- removed link link_gripper
- added link electrode1; visual sphere radius=0.01
- added link electrode2; visual sphere radius=0.01
- added link electrode3; visual sphere radius=0.01
- added link electrode4; visual sphere radius=0.01
- added link electrode5; visual sphere radius=0.01
- added link electrode6; visual sphere radius=0.01
- added link link_straight_gripper, mass 0.0496384234458284; collision mesh filename=package://stretch_description/meshes/link_straight_gripper.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; visual mesh filename=package://stretch_description/meshes/link_straight_gripper.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
- added link link_wrist_pitch, mass 0.0701267146295583; collision mesh filename=package://stretch_description/meshes/link_wrist_pitch.STL; visual mesh filename=package://stretch_description/meshes/link_wrist_pitch.STL
- added link link_wrist_roll, mass 0.00585666394358811; collision mesh filename=package://stretch_description/meshes/link_wrist_roll.STL; visual mesh filename=package://stretch_description/meshes/link_wrist_roll.STL
- added link link_wrist_yaw_bottom, mass 0.0988906816399982; collision mesh filename=package://stretch_description/meshes/link_wrist_yaw_bottom.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; visual mesh filename=package://stretch_description/meshes/link_wrist_yaw_bottom.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
- link link_gripper_finger_left: mass 0.0476207785199474 -> 0.0476207785199479; geometry collision mesh filename=package://stretch_description/meshes/link_gripper_finger_le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; visual mesh filename=package://stretch_description/meshes/link_gripper_finger_le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
- link link_gripper_finger_right: mass 0.0476207785199481 -> 0.047621; geometry collision mesh filename=package://stretch_description/meshes/link_gripper_finger_ri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; visual mesh filename=package://stretch_description/meshes/link_gripper_finger_ri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
- link link_gripper_fingertip_left: mass 0.00382159917455729 -> 0.00382160686584851
- link link_gripper_fingertip_right: mass 0.00382160037319545 -> 0.00382160881468841
- link root_tool: geometry collision mesh filename=package://stretch_description/meshes/Tool1.STL scale=0.01 0.01 0.01; visual mesh filename=package://stretch_description/meshes/Tool1.STL scale=0.01 0.01 0.01
Joints:
- removed joint joint_gripper
- added joint joint_straight_gripper: type fixed, parent link_wrist_roll, child link_straight_gripper, origin xyz=0 0 0.0155 rpy=3.54987407349455E-30 3.24021254484265E-20 -3.14159265358979, axis 0 0 0
- added joint joint_wrist_pitch: type revolute, parent link_wrist_yaw_bottom, child link_wrist_pitch, origin xyz=0 -0.0195500000000002 -0.0247499999999984 rpy=1.5707963267949 -8.12895570882604E-15 -3.14159265358979, axis 0 0 -1, limit lower=-1.57 upper=0.56 effort=100 velocity=1.0
- added joint joint_wrist_roll: type revolute, parent link_wrist_pitch, child link_wrist_roll, origin xyz=-0.0188587444076125 -0.0239999999998942 0.01955 rpy=3.14159265358979 1.5707963267949 0, axis 0 0 1, limit lower=-3.14 upper=3.14 effort=100 velocity=1.0
- added joint joint_wrist_yaw_bottom: type fixed, parent link_wrist_yaw, child link_wrist_yaw_bottom, origin xyz=0 0 0 rpy=-3.14159265358979 1.13367999021379E-14 1.57079632679489, axis 0 0 0
- added joint root_to_electrode1: type prismatic, parent root_tool, child electrode1, origin xyz=-0.055 -0.035 0.01 rpy=0 0 0, axis 0.0 0.0 1.0, limit lower=0.0 upper=1.1 effort=100.0 velocity=1.0
- added joint root_to_electrode2: type prismatic, parent root_tool, child electrode2, origin xyz=-0.055 0.035 0.01 rpy=0 0 0, axis 0.0 0.0 1.0, limit lower=0.0 upper=1.1 effort=100.0 velocity=1.0
- added joint root_to_electrode3: type prismatic, parent root_tool, child electrode3, origin xyz=0 -0.035 0.01 rpy=0 0 0, axis 0.0 0.0 1.0, limit lower=0.0 upper=1.1 effort=100.0 velocity=1.0
- added joint root_to_electrode4: type prismatic, parent root_tool, child electrode4, origin xyz=0 0.035 0.01 rpy=0 0 0, axis 0.0 0.0 1.0, limit lower=0.0 upper=1.1 effort=100.0 velocity=1.0
- added joint root_to_electrode5: type prismatic, parent root_tool, child electrode5, origin xyz=0.055 -0.035 0.01 rpy=0 0 0, axis 0.0 0.0 1.0, limit lower=0.0 upper=1.1 effort=100.0 velocity=1.0
- added joint root_to_electrode6: type prismatic, parent root_tool, child electrode6, origin xyz=0.055 0.035 0.01 rpy=0 0 0, axis 0.0 0.0 1.0, limit lower=0.0 upper=1.1 effort=100.0 velocity=1.0
- joint center_to_tool: origin xyz=0 0 0 rpy=0 0 0 -> xyz=0 0.055 0 rpy=1.57079632679 3.141579 0
- joint joint_grasp_center: origin xyz=-0.205478 0 -0.138154 rpy=0 0 3.141579 -> xyz=0 -0.0125 0.23 rpy=0 0 3.141579; parent link_gripper -> link_straight_gripper
- joint joint_gripper_finger_left: axis 0 0 1 -> 0 0 -1; origin xyz=-0.047231 -0.010151 -0.04679 rpy=2.1762E-15 0.5236 3.1416 -> xyz=0.018599 0.003 0.033689 rpy=1.5708 -1.5708 0; parent link_gripper -> link_straight_gripper
- joint joint_gripper_finger_right: origin xyz=-0.047231 0.010049 -0.04679 rpy=3.1416 -0.5236 1.2943E-15 -> xyz=-0.018599 0.003 0.033689 rpy=1.5708 1.5708 0; parent link_gripper -> link_straight_gripper
- joint joint_gripper_fingertip_left: origin xyz=0.171099 0.014912 0 rpy=-1.5708 -4.774E-15 -2.5545 -> xyz=0.190596948563868 -0.015 0 rpy=1.57079632679496 4.51275387511463E-14 2.60113659715756
- joint joint_gripper_fingertip_right: origin xyz=-0.171099 -0.014912 0 rpy=-1.5708 -2.0539E-15 0.58705 -> xyz=-0.190596948563868 -0.015 0 rpy=-1.57079632679483 -3.43320051448326E-14 0.540456056432235
